File: hardware/ToffeeCam/Camera.kicad_sch (KiCad schematic)
At the start: 25 parts, among them J501 Hirose_FH12-24S-0.5SH(55), U501 TLV74328PDBVR, U502 TLV75512PDBVR

Commit message: Clean schematics
Parts:
- renumbered C502 to C501, C503 to C502, C504 to C503, C505 to C504, C501 to C505, C508 to C506, C509 to C507, C510 to C508, C511 to C509, C506 to C510, C507 to C511, C513 to C512, C514 to C513, C512 to C514
Other:
- moved on the sheet: C505, C510, C511, C514, FB101, J501, R501, R502, R503, R504
