File: hardware/ToffeeCam/PowerSupply.kicad_sch (KiCad schematic)
At the start: 32 parts, among them IC401 TPS26400RHFR, IC402 LDL112PV33R, J401 Messtechnik_AK3001/2-KD-5,0, J401 Wuerth-694108301002

Commit message: Clean schematics
Other:
- moved on the sheet: C306, C401, C402, C403, C404, C405, C406, C407, C408, C410, C411, C412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
