File: hardware/ToffeeCam/ToffeeCam.kicad_pcb (KiCad board)
At the start: 4 copper layers, 156 x 156 mm, 244 parts, among them IC201 W5300, IC301 ADIN1100BCPZ, IC401 TPS26400RHFR, IC402 LDL112PV33R, J201 RJ45, J301 Messtechnik_AK3001/2-KD-5,0, J302 09452812800, J401 Messtechnik_AK3001/2-KD-5,0, J402 Wuerth-694108301002, J501 Hirose_FH12-24S-0.5SH(55), J701 Conn_01x06, J702 USB_B_Micro, P201 RB1-125BAG1A, Q601 AO3401A, SW701 SW_Push, T301 74930000, U301 WE-TVS-82400102, U501 TLV74328PDBVR, U502 TLV75512PDBVR, U701 STM32U575ZITx, U702 WE-TVS-82400102, Y201 7R-25.000MAAQ, Y301 7R-25.000MAAQ, Y701 ABM8G-16.000MHZ-4Y-T3

Commit message: Clean schematics
Parts:
- removed SW701: SW_Push, Button_Switch_THT:SW_Tactile_SPST_Angled_PTS645Vx83-2LFS
- added SW801: SW_Push, Button_Switch_THT:SW_Tactile_SPST_Angled_PTS645Vx83-2LFS, F.Cu at (72.5, 79.3)
- renumbered C218 to C217, C219 to C218, C217 to C219, C223 to C220, C226 to C221, C227 to C222, C228 to C223, C229 to C224, C220 to C225, C221 to C226, C222 to C227, C224 to C228, C225 to C229, C502 to C501, C503 to C502, C504 to C503, C505 to C504, C501 to C505, C508 to C506, C509 to C507, C510 to C508, C511 to C509, C506 to C510, C507 to C511, C513 to C512, C514 to C513, C512 to C514, C722 to C701, C701 to C702, C702 to C703, C703 to C704, C704 to C705, C705 to C706, C723 to C707, C706 to C708, C707 to C709, C708 to C710, C709 to C711, C710 to C712, C711 to C713, C712 to C714, C713 to C715, C714 to C716, C715 to C717, C716 to C718, C717 to C719, C718 to C720, C719 to C721, C720 to C722, C721 to C723, D101 to D801, D102 to D802, D103 to D803, D104 to D804, D105 to D805, D106 to D806, D107 to D807, D108 to D808, FB503 to FB502, FB502 to FB503, FB703 to FB701, FB704 to FB702, FB705 to FB703, FB701 to FB704, FB702 to FB705, H101 to H801, H102 to H802, H103 to H803, H104 to H804, H105 to H805, H106 to H806, H107 to H807, H108 to H808, J702 to J701, J701 to J702, R212 to R210, R210 to R211, R211 to R212, R705 to R701, R706 to R702, R707 to R703, R701 to R704, R702 to R705, R703 to R706, R704 to R707, R101 to R801, R102 to R802, R103 to R803, R104 to R804, R105 to R805, R106 to R806, R107 to R807, R108 to R808, R109 to R809, R110 to R810, U702 to U701, U701 to U702
Connections:
- U702 pad 47: Net-(U701-PB1) -> PUSHBUTTON
Routing:
- net PUSHBUTTON: track 0.00 -> 45.7 mm, vias 0 -> 1
- net Net-(U701-PB1): track 45.7 -> 0.00 mm, vias 1 -> 0
