File: hardware/ToffeeCam/ToffeeCam.kicad_sch (KiCad schematic)
At the start: 26 parts

Commit message: Clean schematics
Parts:
- removed D101, D103, D104, D107, D108, D302, D303: LED, LED_SMD:LED_0805_2012Metric, symbol Device:LED
- removed D102: BZX84Cxx, Package_TO_SOT_SMD:SOT-23, symbol Diode:BZX84Cxx
- removed H101, H102, H107, H108: MountingHole, Project_Speciific_Mechanical:MountingHole-10mm, symbol Mechanical:MountingHole
- removed H103, H104, H105, H106: MountingHole, Project_Speciific_Mechanical:MountingHole_2.5mm, symbol Mechanical:MountingHole
- removed R101, R104, R109, R110: 330R, Resistor_SMD:R_0603_1608Metric, symbol Device:R
- removed R102, R103, R308, R311: 4k7, Resistor_SMD:R_0603_1608Metric, symbol Device:R
- removed R309, R310: 100, Resistor_SMD:R_0603_1608Metric, symbol Device:R
Other:
- added sheet Panel (Panel.kicad_sch)
