File: hardware/ToffeeCam/MCU.kicad_sch (KiCad schematic)
At the start: 45 parts, among them J101 USB_B_Micro, J201 Conn_01x06, SW701 SW_Push, U1 STM32U575ZITx, U101 WE-TVS-82400102, Y701 ABM8G-16.000MHZ-4Y-T3

Commit message: Clean schematics
Parts:
- removed SW701: SW_Push, Button_Switch_THT:SW_Tactile_SPST_Angled_PTS645Vx83-2LFS, symbol Switch:SW_Push
- renumbered C701 to C702, C702 to C703, C703 to C704, C704 to C705, C705 to C706, C706 to C708, C707 to C709, C708 to C710, C709 to C711, C710 to C712, C711 to C713, C712 to C714, C713 to C715, C714 to C716, C715 to C717, C716 to C718, C717 to C719, C718 to C720, C719 to C721
Connections:
- net PUSHBUTTON: now reaches U1.47 (PB1)
Other:
- moved on the sheet: C111, C112, C301, C302, C702, C703, C704, C705, C706, C708, C709, C710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

Commit message: Docs up to date
Parts:
- F101: value Polyfuse_Small -> 0.5A
- FB101: value HH-1M1608-221JT -> HH-1M1608-121JT
- J101: value USB_B_Micro -> Molex-105133-0001
Changed lines of the file:
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@@
       (effects (font (size 1.27 1.27)))
     )
-    (property "Value" "HH-1M1608-221JT" (at 280.67 113.03 90)
+    (property "Value" "HH-1M1608-121JT" (at 280.67 113.03 90)
       (effects (font (size 0.6 0.6)))
     )
@@
       (effects (font (size 1.27 1.27)))
     )
-    (property "Value" "HH-1M1608-221JT" (at 279.4 105.41 90)
+    (property "Value" "HH-1M1608-121JT" (at 279.4 105.41 90)
       (effects (font (size 0.6 0.6)))
     )
@@
       (effects (font (size 1.27 1.27)))
     )
-    (property "Value" "Polyfuse_Small" (at 99.06 261.62 90)
-      (effects (font (size 0.6 0.6)))
+    (property "Value" "0.5A" (at 97.79 261.62 90)
+      (effects (font (size 1.27 1.27)))
     )
     (property "Footprint" "Fuse:Fuse_1812_4532Metric" (at 101.6 266.7 0)
@@
       (effects (font (size 1.27 1.27)) (justify left))
     )
-    (property "Value" "USB_B_Micro" (at 107.6452 235.712 90)
+    (property "Value" "Molex-105133-0001" (at 107.6452 235.712 90)
       (effects (font (size 0.6 0.6)) (justify left))
     )
