File: hardware/ToffeeCam/Panel.kicad_sch (KiCad schematic)
At the start: 27 parts, among them SW701 SW_Push

Commit message: Docs up to date
Parts:
- D102: value BZX84Cxx -> BZX84C12
Changed lines of the file:
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@@
       (effects (font (size 1.27 1.27)) (justify left))
     )
-    (property "Value" "BZX84Cxx" (at 95.25 97.79 90)
+    (property "Value" "BZX84C12" (at 95.25 97.79 90)
       (effects (font (size 1.27 1.27)) (justify left))
     )
