File: hardware/ToffeeCam/Wiznet-W5300.kicad_sch (KiCad schematic)
At the start: 48 parts, among them IC1 W5300, J201 RJ45, P201 RB1-125BAG1A, Y301 7R-25.000MAAQ

Commit message: Clean schematics
Parts:
- renumbered C218 to C217, C219 to C218, C217 to C219, C227 to C222, C228 to C223, C229 to C224, C220 to C225, C221 to C226, C222 to C227, C224 to C228, C225 to C229, R212 to R210, R210 to R211, R211 to R212
Other:
- note added: "Transformer variant"
- note added: "Transformerless variant"
- moved on the sheet: C213, C219, C225, C226, C227, C228, C229, J201, P201, R211, R212

Commit message: Docs up to date
Parts:
- Y301: value 7R-25.000MAAQ -> WE-830108212509
Changed lines of the file:
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@@
   (symbol (lib_id "Device:Crystal_GND24_Small") (at 205.74 238.76 270) (unit 1)
     (in_bom yes) (on_board yes) (dnp no)
-    (property "Reference" "Y301" (at 203.835 235.585 90)
+    (property "Reference" "Y301" (at 203.2 234.95 90)
       (effects (font (size 1.27 1.27)))
     )
-    (property "Value" "7R-25.000MAAQ" (at 209.55 236.22 90)
+    (property "Value" "WE-830108212509" (at 210.82 236.22 90)
       (effects (font (size 0.6 0.6)))
     )
