File: hardware/ToffeeCam/Ethernet-10BASE-T1L.kicad_sch (KiCad schematic)
At the start: 51 parts, among them IC301 ADIN1100BCPZ, J301 09452812800, J403 Messtechnik_AK3001/2-KD-5,0, T301 74930000, U302 WE-TVS-82400102, Y301 7R-25.000MAAQ

Commit message: Clean schematics
Changed lines of the file:
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@@
   (symbol (lib_id "Project_Specific_AnalogDevices:ADIN1100BCPZ") (at 143.51 123.19 90) (unit 1)
     (in_bom yes) (on_board yes) (dnp no)
-    (property "Reference" "IC301" (at 138.43 121.92 90)
+    (property "Reference" "IC301" (at 140.97 124.46 90)
       (effects (font (size 3.81 3.81)))
     )

Commit message: Docs up to date
Parts:
- C301, C302: value 16p -> 13p
- F301, F302: value Fuse -> 0.2A
- Y301: value 7R-25.000MAAQ -> WE-830108212509
Changed lines of the file:
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@@
       (effects (font (size 1.27 1.27)))
     )
-    (property "Value" "Fuse" (at 331.47 130.81 90)
+    (property "Value" "0.2A" (at 331.47 130.81 90)
       (effects (font (size 1.27 1.27)))
     )
@@
       (effects (font (size 1.27 1.27)))
     )
-    (property "Value" "Fuse" (at 331.47 155.575 90)
+    (property "Value" "0.2A" (at 331.47 155.575 90)
       (effects (font (size 1.27 1.27)))
     )
@@
   (symbol (lib_id "Device:C") (at 162.56 191.77 270) (unit 1)
     (in_bom yes) (on_board yes) (dnp no) (fields_autoplaced)
-    (property "Reference" "C301" (at 161.2899 187.96 0)
-      (effects (font (size 1.27 1.27)) (justify right))
-    )
-    (property "Value" "16p" (at 163.8299 187.96 0)
-      (effects (font (size 0.6 0.6)) (justify right))
+    (property "Reference" "C301" (at 162.56 185.42 90)
+      (effects (font (size 1.27 1.27)))
+    )
+    (property "Value" "13p" (at 162.56 187.96 90)
+      (effects (font (size 0.6 0.6)))
     )
     (property "Footprint" "Capacitor_SMD:C_0402_1005Metric" (at 158.75 192.7352 0)
@@
   (symbol (lib_id "Device:C") (at 162.56 179.07 90) (unit 1)
     (in_bom yes) (on_board yes) (dnp no) (fields_autoplaced)
-    (property "Reference" "C302" (at 161.2899 175.26 0)
-      (effects (font (size 1.27 1.27)) (justify left))
-    )
-    (property "Value" "16p" (at 163.8299 175.26 0)
-      (effects (font (size 0.6 0.6)) (justify left))
+    (property "Reference" "C302" (at 162.56 172.72 90)
+      (effects (font (size 1.27 1.27)))
+    )
+    (property "Value" "13p" (at 162.56 175.26 90)
+      (effects (font (size 0.6 0.6)))
     )
     (property "Footprint" "Capacitor_SMD:C_0402_1005Metric" (at 166.37 178.1048 0)
@@
       (effects (font (size 1.27 1.27)))
     )
-    (property "Value" "7R-25.000MAAQ" (at 148.59 179.07 90)
-      (effects (font (size 0.6 0.6)))
-    )
+    (property "Value" "WE-830108212509" (at 148.59 179.07 90)
+      (effects (font (size 0.6 0.6)))
+    )

Commit message: Docs for Wiznet's contest
Parts:
- R312: value 4k7 -> NP
Changed lines of the file:
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@@
       (effects (font (size 1.27 1.27)))
     )
-    (property "Value" "4k7" (at 125.73 80.01 90)
+    (property "Value" "NP" (at 125.73 80.01 90)
       (effects (font (size 1.27 1.27)))
     )
@@
       (effects (font (size 1.27 1.27)))
     )
-    (property "Value" "4k7" (at 114.3 80.01 90)
+    (property "Value" "NP" (at 114.3 80.01 90)
       (effects (font (size 1.27 1.27)))
     )
@@
       (effects (font (size 1.27 1.27)))
     )
-    (property "Value" "4k7" (at 93.98 99.06 90)
-      (effects (font (size 1.27 1.27)))
-    )
+    (property "Value" "NP" (at 93.98 99.06 90)
+      (effects (font (size 1.27 1.27)))
+    )
